File: MCP73213T_2S.kicad_pcb (KiCad board)
At the start: 2 copper layers, 34 x 11 mm, 16 parts, among them J1 Conn_01x10, J2 Conn_01x10, J3 Conn_01x01_Female, J4 Conn_01x01_Female, J5 Conn_01x01_Female, J6 Conn_01x01_Female, U1 MCP73213T

Commit message: added power module
Parts:
- added U1: TLVM13620RDHR, TI_POWER_MODULE:TLVM13620RDHR, F.Cu at (142.1, 104.2)
- moved C2 16.6 mm to (133.4, 91.0)
- moved C3 15.2 mm to (139.3, 90.5)
- renumbered R4 to R1, R5 to R2, U1 to U2
Connections:
- J1 pad 6: /STAT_3 -> Net-(J1-Pad6)
- J1 pad 7: /STAT_2 -> Net-(J1-Pad7)
- J1 pad 8: /STAT_1 -> Net-(J1-Pad8)
- J2 pad 3: /STAT_1 -> Net-(J1-Pad8)
- J2 pad 4: /STAT_2 -> Net-(J1-Pad7)
- J2 pad 5: /STAT_3 -> Net-(J1-Pad6)
Routing:
- net Net-(J1-Pad8): track 0.00 -> 7.56 mm, vias 0 -> 1
- net /STAT_1: track 7.56 -> 0.00 mm, vias 1 -> 0
- net GND: vias 4 -> 2
